File: Electrics/Catlift.sch (KiCad schematic (older format))
At the start: 1 part

Commit message: KiCAD Update to 5.1.4, some sketches
Parts:
- removed M?: Motor_Servo, symbol Motor_Servo
- added M?: Motor_DC, symbol Motor:Motor_DC
- added M?: Motor_Servo, symbol Motor:Motor_Servo
- added R?: A1050, OptoDevice:R_LDR_D6.4mm_P3.4mm_Vertical, symbol Sensor_Optical:A1050
Changed lines of the file:
@@
-EESchema Schematic File Version 2
-LIBS:power
-LIBS:device
-LIBS:switches
-LIBS:relays
-LIBS:motors
-LIBS:transistors
-LIBS:conn
-LIBS:linear
-LIBS:regul
-LIBS:74xx
-LIBS:cmos4000
-LIBS:adc-dac
-LIBS:memory
-LIBS:xilinx
-LIBS:microcontrollers
-LIBS:dsp
-LIBS:microchip
-LIBS:analog_switches
-LIBS:motorola
-LIBS:texas
-LIBS:intel
-LIBS:audio
-LIBS:interface
-LIBS:digital-audio
-LIBS:philips
-LIBS:display
-LIBS:cypress
-LIBS:siliconi
-LIBS:opto
-LIBS:atmel
-LIBS:contrib
-LIBS:valves
-LIBS:Arduino_Uno_R3_From_Scratch-cache
-EELAYER 25 0
+EESchema Schematic File Version 4
+LIBS:Catlift-cache
+EELAYER 30 0
 EELAYER END
 $Descr A4 11693 8268
@@
 Comment4 ""
 $EndDescr
-$Comp
-L +15V #PWR?
-U 1 1 5D6EB84F
-P -2400 -2450
-F 0 "#PWR?" H -2400 -2600 50  0001 C CNN
-F 1 "+15V" H -2400 -2310 50  0000 C CNN
-F 2 "" H -2400 -2450 50  0001 C CNN
-F 3 "" H -2400 -2450 50  0001 C CNN
-	1    -2400 -2450
-	1    0    0    -1
-$EndComp
-$Comp
-L +15V #PWR?
-U 1 1 5D6EB863
-P 1800 1900
-F 0 "#PWR?" H 1800 1750 50  0001 C CNN
-F 1 "+15V" H 1800 2040 50  0000 C CNN
-F 2 "" H 1800 1900 50  0001 C CNN
-F 3 "" H 1800 1900 50  0001 C CNN
-	1    1800 1900
-	1    0    0    -1
-$EndComp
-$Comp
-L Motor_Servo M?
-U 1 1 5D6EB884
-P 3200 2250
-F 0 "M?" H 3000 2425 50  0000 L CNN
-F 1 "Motor_Servo" H 3000 2090 50  0000 L TNN
-F 2 "" H 3200 2060 50  0001 C CNN
-F 3 "" H 3200 2060 50  0001 C CNN
-	1    3200 2250
-	1    0    0    -1
-$EndComp
 $Sheet
 S 2050 1400 1500 1500
@@
 	7050 2700 7550 2700
 Wire Wire Line
-	7550 2850 7050 2850
+	7550 2850 7300 2850
 Wire Wire Line
 	7050 3000 7550 3000
@@
 	7300 1750 7300 2850
 Connection ~ 7300 2850
+Wire Wire Line
+	7300 2850 7050 2850
+$Comp
+L Motor:Motor_DC M?
+U 1 1 5D6ED75A
+P 14600 1850
+F 0 "M?" H 14758 1846 50  0000 L CNN
+F 1 "Motor_DC" H 14758 1755 50  0000 L CNN
+F 2 "" H 14600 1760 50  0001 C CNN
+F 3 "~" H 14600 1760 50  0001 C CNN
+	1    14600 1850
+	1    0    0    -1
+$EndComp
+$Comp
+L Motor:Motor_Servo M?
+U 1 1 5D6EDF11
+P 14650 4050
+F 0 "M?" H 14982 4115 50  0000 L CNN
+F 1 "Motor_Servo" H 14982 4024 50  0000 L CNN
+F 2 "" H 14650 3860 50  0001 C CNN
+F 3 "http://forums.parallax.com/uploads/attachments/46831/74481.png" H 14650 3860 50  0001 C CNN
+	1    14650 4050
+	1    0    0    -1
+$EndComp
+$Comp
+L Sensor_Optical:A1050 R?
+U 1 1 5D6EEF5A
+P 14350 5350
+F 0 "R?" H 14420 5396 50  0000 L CNN
+F 1 "A1050" H 14420 5305 50  0000 L CNN
+F 2 "OptoDevice:R_LDR_D6.4mm_P3.4mm_Vertical" V 14525 5350 50  0001 C CNN
+F 3 "http://cdn-reichelt.de/documents/datenblatt/A500/A106012.pdf" H 14350 5300 50  0001 C CNN
+	1    14350 5350
+	1    0    0    -1
+$EndComp
 $EndSCHEMATC
